File: reference_design/G76 Mini.kicad_pcb (KiCad board)
At the start: 4 copper layers, 49.3 x 72.3 mm, 28 parts, among them J1 Conn_02x16_Odd_Even, J2 Conn_02x05_Odd_Even, J3 DB15_Female_HighDensity, U1 EPM240T100, U2 CY7C1018DV33, X1 50MHz

Commit message: Fix CE line on RAM
Parts:
- J2: value Conn_02x05_Odd_Even -> JTAG
- U2: value CY7C1018DV33 -> CY7C1018DV33-10VXI
Connections:
- U2 pad 5: /~{VRAM_CE} -> GND
Changed lines of the file:
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@@
   (net 96 "/VRAM_A16")
   (net 97 "unconnected-(U1-Pad100)")
-  (net 98 "/~{VRAM_CE}")
-  (net 99 "unconnected-(X1-Pad1)")
+  (net 98 "unconnected-(X1-Pad1)")
   (footprint "Resistor_SMD:R_1206_3216Metric_Pad1.30x1.75mm_HandSolder" (layer "F.Cu")
     (at 94.615 63.474 90)
@@
     (fp_arc (start 16.97 1.19) (mid 16.867487 1.437487) (end 16.62 1.54) (layer "F.Fab") (width 0.1))
     (pad "1" thru_hole rect (at 0 0 90) (size 1.6 1.6) (drill 0.8) (layers *.Cu *.Mask)
-      (net 99 "unconnected-(X1-Pad1)") (pinfunction "NC") (pintype "no_connect"))
+      (net 98 "unconnected-(X1-Pad1)") (pinfunction "NC") (pintype "no_connect"))
     (pad "7" thru_hole circle (at 15.24 0 90) (size 1.6 1.6) (drill 0.8) (layers *.Cu *.Mask)
       (net 2 "GND") (pinfunction "GND") (pintype "power_in"))
@@
       (effects (font (size 1 1) (thickness 0.15)))
     )
-    (fp_text value "CY7C1018DV33" (at 0 0 90) (layer "F.Fab")
+    (fp_text value "CY7C1018DV33-10VXI" (at 0 0 90) (layer "F.Fab")
       (effects (font (size 1 1) (thickness 0.15)))
     )
@@
       (net 83 "/VRAM_A3") (pinfunction "A3") (pintype "input"))
     (pad "5" smd rect (at -4.445 3.81 270) (size 0.45 2.2) (layers "F.Cu" "F.Paste" "F.Mask")
-      (net 98 "/~{VRAM_CE}") (pinfunction "~{CE}") (pintype "input"))
+      (net 2 "GND") (pinfunction "~{CE}") (pintype "input"))
     (pad "6" smd rect (at -3.175 3.81 270) (size 0.45 2.2) (layers "F.Cu" "F.Paste" "F.Mask")
       (net 67 "/VRAM_D0") (pinfunction "Q0") (pintype "tri_state"))
@@
       (effects (font (size 1 1) (thickness 0.15)))
     )
-    (fp_text value "Conn_02x05_Odd_Even" (at 1.27 12.49) (layer "F.Fab")
-      (effects (font (size 1 1) (thickness 0.15)))
-    )
+    (fp_text value "JTAG" (at 1.27 12.49) (layer "F.Fab")
+      (effects (font (size 1 1) (thickness 0.15)))
+    )
